File: RoboRG-eda.kicad_pcb (KiCad board)
At the start: 4 copper layers, 50 x 100 mm, 84 parts, among them J1 USB_C_Receptacle_USB2.0, J2 AudioJack3_Switch, J3 connector-pan, J4 connector-tilt, J5 connector-other, J6 USB_C_Receptacle_USB2.0, J7 SWD, J8 USART, J9 Barrel_Jack_Switch, Q1 Q_PNP_BEC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

Commit message: Fix version number on the silkscreen
Other:
- board text added: "1.0.2"
- board text removed: "1.0.1"
Changed lines of the file:
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@@
     (34 B.Paste user)
     (35 F.Paste user)
-    (36 B.SilkS user hide)
+    (36 B.SilkS user)
     (37 F.SilkS user)
     (38 B.Mask user)
@@
     (effects (font (size 1.5 1.5) (thickness 0.3)) (justify mirror))
   )
-  (gr_text 1.0.1 (at 123.9 77.75 270) (layer B.SilkS)
+  (gr_text 1.0.2 (at 123.9 77.75 270) (layer B.SilkS)
     (effects (font (size 2 2) (thickness 0.3)) (justify mirror))
   )
